Commit message: update a1 urdf; a working wbc init test program

File: src/legged_ctrl/urdf/a1_description/urdf/a1.urdf (robot description, URDF)
Before this commit: robot a1_description, 23 links, 22 joints
Links:
- removed link FL_calf
- removed link FL_foot
- removed link FL_hip
- removed link FL_thigh
- removed link FL_thigh_shoulder
- removed link FR_calf
- removed link FR_foot
- removed link FR_hip
- removed link FR_thigh
- removed link FR_thigh_shoulder
- removed link RL_calf
- removed link RL_foot
- removed link RL_hip
- removed link RL_thigh
- removed link RL_thigh_shoulder
- removed link RR_calf
- removed link RR_foot
- removed link RR_hip
- removed link RR_thigh
- removed link RR_thigh_shoulder
- removed link imu_link
- removed link trunk
- added link LF_FOOT, mass 0.06; collision sphere radius=0.02; visual sphere radius=0.01
- added link LF_calf, mass 0.151; collision box size=0.2 0.016 0.016; visual mesh filename=package://unitree_description/meshes/a1/calf.dae scale=1 1 1
- added link LF_hip, mass 0.595; collision cylinder length=0.04 radius=0.046; visual mesh filename=package://unitree_description/meshes/a1/hip.dae scale=1 1 1
- added link LF_thigh, mass 0.888; collision box size=0.2 0.0245 0.034; collision cylinder length=0.032 radius=0.041
- added link LH_FOOT, mass 0.06; collision sphere radius=0.02; visual sphere radius=0.01
- added link LH_calf, mass 0.151; collision box size=0.2 0.016 0.016; visual mesh filename=package://unitree_description/meshes/a1/calf.dae scale=1 1 1
- added link LH_hip, mass 0.595; collision cylinder length=0.04 radius=0.046; visual mesh filename=package://unitree_description/meshes/a1/hip.dae scale=1 1 1
- added link LH_thigh, mass 0.888; collision box size=0.2 0.0245 0.034; collision cylinder length=0.032 radius=0.041
- added link RF_FOOT, mass 0.06; collision sphere radius=0.02; visual sphere radius=0.01
- added link RF_calf, mass 0.151; collision box size=0.2 0.016 0.016; visual mesh filename=package://unitree_description/meshes/a1/calf.dae scale=1 1 1
- added link RF_hip, mass 0.595; collision cylinder length=0.04 radius=0.046; visual mesh filename=package://unitree_description/meshes/a1/hip.dae scale=1 1 1
- added link RF_thigh, mass 0.888; collision box size=0.2 0.0245 0.034; collision cylinder length=0.032 radius=0.041
- added link RH_FOOT, mass 0.06; collision sphere radius=0.02; visual sphere radius=0.01
- added link RH_calf, mass 0.151; collision box size=0.2 0.016 0.016; visual mesh filename=package://unitree_description/meshes/a1/calf.dae scale=1 1 1
- added link RH_hip, mass 0.595; collision cylinder length=0.04 radius=0.046; visual mesh filename=package://unitree_description/meshes/a1/hip.dae scale=1 1 1
- added link RH_thigh, mass 0.888; collision box size=0.2 0.0245 0.034; collision cylinder length=0.032 radius=0.041
- added link unitree_imu, mass 0.01; visual box size=0.015 0.015 0.004
- link base: mass None -> 6.0; geometry collision box size=0.267 0.194 0.114; visual mesh filename=package://unitree_description/meshes/a1/trunk.dae scale=1 1 1
Joints:
- removed joint FL_calf_joint
- removed joint FL_foot_fixed
- removed joint FL_hip_fixed
- removed joint FL_hip_joint
- removed joint FL_thigh_joint
- removed joint FR_calf_joint
- removed joint FR_foot_fixed
- removed joint FR_hip_fixed
- removed joint FR_hip_joint
- removed joint FR_thigh_joint
- removed joint RL_calf_joint
- removed joint RL_foot_fixed
- removed joint RL_hip_fixed
- removed joint RL_hip_joint
- removed joint RL_thigh_joint
- removed joint RR_calf_joint
- removed joint RR_foot_fixed
- removed joint RR_hip_fixed
- removed joint RR_hip_joint
- removed joint RR_thigh_joint
- removed joint floating_base
- removed joint imu_joint
- added joint LF_HAA: type revolute, parent base, child LF_hip, origin xyz=0.1805 0.047 0 rpy=0 0 0, axis 1 0 0, limit lower=-0.8028514559173915 upper=0.8028514559173915 effort=33.5 velocity=21
- added joint LF_HFE: type revolute, parent LF_hip, child LF_thigh, origin xyz=0 0.0838 0 rpy=0 0 0, axis 0 1 0, limit lower=-1.0471975511965976 upper=4.1887902047863905 effort=33.5 velocity=21
- added joint LF_KFE: type revolute, parent LF_thigh, child LF_calf, origin xyz=0 0 -0.2 rpy=0 0 0, axis 0 1 0, limit lower=-2.6965336943312392 upper=-0.9162978572970231 effort=33.5 velocity=21
- added joint LF_foot_fixed: type fixed, parent LF_calf, child LF_FOOT, origin xyz=0 0 -0.2 rpy=0 0 0
- added joint LH_HAA: type revolute, parent base, child LH_hip, origin xyz=-0.1805 0.047 0 rpy=0 0 0, axis 1 0 0, limit lower=-0.8028514559173915 upper=0.8028514559173915 effort=33.5 velocity=21
- added joint LH_HFE: type revolute, parent LH_hip, child LH_thigh, origin xyz=0 0.0838 0 rpy=0 0 0, axis 0 1 0, limit lower=-1.0471975511965976 upper=4.1887902047863905 effort=33.5 velocity=21
- added joint LH_KFE: type revolute, parent LH_thigh, child LH_calf, origin xyz=0 0 -0.2 rpy=0 0 0, axis 0 1 0, limit lower=-2.6965336943312392 upper=-0.9162978572970231 effort=33.5 velocity=21
- added joint LH_foot_fixed: type fixed, parent LH_calf, child LH_FOOT, origin xyz=0 0 -0.2 rpy=0 0 0
- added joint RF_HAA: type revolute, parent base, child RF_hip, origin xyz=0.1805 -0.047 0 rpy=0 0 0, axis 1 0 0, limit lower=-0.8028514559173915 upper=0.8028514559173915 effort=33.5 velocity=21
- added joint RF_HFE: type revolute, parent RF_hip, child RF_thigh, origin xyz=0 -0.0838 0 rpy=0 0 0, axis 0 1 0, limit lower=-1.0471975511965976 upper=4.1887902047863905 effort=33.5 velocity=21
- added joint RF_KFE: type revolute, parent RF_thigh, child RF_calf, origin xyz=0 0 -0.2 rpy=0 0 0, axis 0 1 0, limit lower=-2.6965336943312392 upper=-0.9162978572970231 effort=33.5 velocity=21
- added joint RF_foot_fixed: type fixed, parent RF_calf, child RF_FOOT, origin xyz=0 0 -0.2 rpy=0 0 0
- added joint RH_HAA: type revolute, parent base, child RH_hip, origin xyz=-0.1805 -0.047 0 rpy=0 0 0, axis 1 0 0, limit lower=-0.8028514559173915 upper=0.8028514559173915 effort=33.5 velocity=21
- added joint RH_HFE: type revolute, parent RH_hip, child RH_thigh, origin xyz=0 -0.0838 0 rpy=0 0 0, axis 0 1 0, limit lower=-1.0471975511965976 upper=4.1887902047863905 effort=33.5 velocity=21
- added joint RH_KFE: type revolute, parent RH_thigh, child RH_calf, origin xyz=0 0 -0.2 rpy=0 0 0, axis 0 1 0, limit lower=-2.6965336943312392 upper=-0.9162978572970231 effort=33.5 velocity=21
- added joint RH_foot_fixed: type fixed, parent RH_calf, child RH_FOOT, origin xyz=0 0 -0.2 rpy=0 0 0
- added joint unitree_imu_joint: type fixed, parent base, child unitree_imu, origin xyz=0. 0. 0. rpy=0. 0. 0.
